File: KiCAD_schematics/Wiring.kicad_sch (KiCad schematic)
At the start: 7 parts, among them J2 MP1583EN Buck Converter, J3 Conn_01x04, K2 SANYOU_SRD_Form_C, M1 Motor_DC, U1 HX711

Commit message: Mass Changes
Forgot to commit as changes were made. SSD1306 display logic has been added.
Parts:
- added C1: 100nF, symbol Device:C
- added C2: 10uF, symbol Device:C_Polarized
- added R1: 100, symbol Device:R
Connections:
- net at A1.19 (GPIO14): now also R1.1; no longer U1.11 (PD_SCK)
- net at A1.33 (AGND), Brd1.1 (GND), J2.Vout- (Pin_5)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: now also C1.2, C2.2
- net at U1.6 (VBG): now also A1.36 (3V3), Brd1.2 (VCC), C1.1, C2.1
- net at A1.39 (VSYS), J2.Vout+ (Pin_7), K2.VCC: no longer Brd1.2 (VCC)
- new net: R1.2, U1.11 (PD_SCK)
